File: Hardware/Qwiic RFID - IDXXLA.sch (EAGLE design)
At the start: 35 parts, among them J3 PTH, J8 AVR_SPI_PROG_3X2TESTPOINTS, Q1 600mA/40V, U1 ATTINY84-ARDUINO, U2 ID-12/20SMD

Commit message: Updates general trace layout, moves interrupt jumper to upper right, moves stat LED to TOP layer parallel with PWR LED
* Adds SparkFun Flame and removes SparkX references
* Changes version
* Updates text to vector in schematic.
* Updates Qwiic_RFID silk and power LED to something larger.
Parts:
- removed U$4: SPARKX-LOGO3, SparkX:SPARKX-LOGO3
- added LOGO2: SFE_LOGO_FLAME.1_INCH, SparkFun-Aesthetics:SFE_LOGO_FLAME.1_INCH
Other:
- note added: "7-Bit Unshifted I2C Address Open Jumper (Default): 0x7D Closed Jumper: 0x7C Software configurable"
- note added: "Elias Santsitevan"
- note added: "v10"
- note removed: "7-Bit Unshifted I2C Address Open Jumper (Default): 0x7D Closed Jumper: 0x7C Software configurable as well"
- note removed: "Elias Santistevan"
- note removed: "X02"

Commit message: Adds better SparkFun silk, changes text to vector, and updates product name silk
Parts:
- LOGO2: value SFE_LOGO_FLAME.1_INCH -> SFE_LOGO_NAME.1_INCH; device SparkFun-Aesthetics:SFE_LOGO_FLAME.1_INCH -> SparkFun-Aesthetics:SFE_LOGO_NAME.1_INCH
Other:
- note added: "VCC: 3.3V Only"
Changed lines of the file:
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@@
 <part name="SUPPLY13" library="SparkFun-PowerSymbols" deviceset="3.3V" device=""/>
 <part name="GND11" library="SparkFun-PowerSymbols" deviceset="GND" device=""/>
-<part name="LOGO2" library="SparkFun-Aesthetics" deviceset="SFE_LOGO_FLAME" device=".1_INCH"/>
+<part name="LOGO2" library="SparkFun-Aesthetics" deviceset="SFE_LOGO_NAME" device=".1_INCH"/>
 </parts>
 <sheets>
@@
 <text x="238.76" y="7.62" size="2.54" layer="94" font="vector">v10</text>
 <text x="162.56" y="7.62" size="2.54" layer="94" font="vector">Elias Santsitevan</text>
+<text x="33.02" y="137.16" size="1.778" layer="97" font="vector">VCC: 3.3V Only</text>
 </plain>
 <instances>
@@
 <attribute name="VALUE" x="15.24" y="108.966" size="1.778" layer="96" font="vector" align="top-center"/>
 </instance>
-<instance part="LOGO2" gate="G$1" x="214.884" y="38.862" smashed="yes"/>
+<instance part="LOGO2" gate="G$1" x="165.1" y="33.02" smashed="yes"/>
 </instances>
 <busses>

Commit message: Changes sparkFun logo to sparkFun + flame logo, adds dimensions for standoffs
Parts:
- removed LOGO2: SFE_LOGO_NAME.1_INCH, SparkFun-Aesthetics:SFE_LOGO_NAME.1_INCH
- added LOGO3: SFE_LOGO_NAME_FLAME.1_INCH, SparkFun-Aesthetics:SFE_LOGO_NAME_FLAME.1_INCH
Changed lines of the file:
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@@
 <part name="SUPPLY13" library="SparkFun-PowerSymbols" deviceset="3.3V" device=""/>
 <part name="GND11" library="SparkFun-PowerSymbols" deviceset="GND" device=""/>
-<part name="LOGO2" library="SparkFun-Aesthetics" deviceset="SFE_LOGO_NAME" device=".1_INCH"/>
+<part name="LOGO3" library="SparkFun-Aesthetics" deviceset="SFE_LOGO_NAME_FLAME" device=".1_INCH"/>
 </parts>
 <sheets>
@@
 <attribute name="VALUE" x="15.24" y="108.966" size="1.778" layer="96" font="vector" align="top-center"/>
 </instance>
-<instance part="LOGO2" gate="G$1" x="165.1" y="33.02" smashed="yes"/>
+<instance part="LOGO3" gate="G$1" x="167.64" y="33.02" smashed="yes"/>
 </instances>
 <busses>

Commit message: Update Schematic to Reflect I2C Address Change
Other:
- note added: "7-Bit Unshifted I2C Address Open Jumper (Default): 0x13 Closed Jumper: 0x14 Software configurable"
- note removed: "7-Bit Unshifted I2C Address Open Jumper (Default): 0x7D Closed Jumper: 0x7C Software configurable"
Changed lines of the file:
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@@
 <?xml version="1.0" encoding="utf-8"?>
 <!DOCTYPE eagle SYSTEM "eagle.dtd">
-<eagle version="9.2.1">
+<eagle version="9.6.2">
 <drawing>
 <settings>
@@
 <wire x1="81.28" y1="83.82" x2="81.28" y2="0" width="0.2032" layer="97" style="shortdash"/>
 <text x="83.058" y="91.44" size="1.778" layer="97" font="vector">7-Bit Unshifted I2C Address
-Open Jumper (Default): 0x7D
-Closed Jumper: 0x7C
+Open Jumper (Default): 0x13
+Closed Jumper: 0x14
 Software configurable </text>
 <text x="129.54" y="35.56" size="1.778" layer="97" font="vector">Cut Buzzer Jumper
